Commit message: feat: update assets

File: xmimic/humanoidverse/asset/objects/basketball/ball.urdf (robot description, URDF)
Before this commit: robot ball, 1 links, 0 joints
Links:
- link ball: geometry collision sphere radius=0.123; visual sphere radius=0.123

Commit message: feat: multi-skill sampling weight

File: xmimic/humanoidverse/asset/objects/basketball/ball.urdf (robot description, URDF)
Before this commit: robot ball, 1 links, 0 joints
Links:
- link ball: geometry collision sphere radius=0.12; visual sphere radius=0.12

Commit message: feat: update params, fix rotation reward

File: xmimic/humanoidverse/asset/objects/basketball/ball.urdf (robot description, URDF)
Before this commit: robot ball, 1 links, 0 joints
Links:
- link ball: mass 0.5 -> 0.6
