Commit message: feat: update asset

File: xmimic/humanoidverse/asset/robots/g1/g1_29dof_mode16_bb.urdf (robot description, URDF)
Before this commit: robot g1_29dof_mode15_w_hand, 39 links, 38 joints
Links:
- link left_rubber_hand: geometry collision mesh filename=meshes/bowl_convex/left/hull_000.obj scale=0.001 0.001 0.001; collision mesh filename=meshes/bowl_convex/left/hull_001.obj scale=0.001 0.001 0.001
- link right_rubber_hand: geometry collision mesh filename=meshes/bowl_convex/right/hull_000.obj scale=0.001 0.001 0.001; collision mesh filename=meshes/bowl_convex/right/hull_001.obj scale=0.001 0.001 0.001
